File: HeartPCBGift.kicad_pcb (KiCad board)
At the start: 2 copper layers, 80.7 x 71.6 mm, 68 parts, among them J1 Conn_02x03_Odd_Even, U1 ATMEGA32U4-AU, U2 MF-MSMF050-2, X1 X322516MLB4SI

Commit message: Removed useless files
Parts:
- removed the G*** at (139.0, 84.0)
Other:
- board text added: "A MESSAGE TO THE GIFT RECIPIENT"
- board text added: "XX.XX.XXXXX (a date if wanted)"
- board text removed: "VI.XI.MMXXVI"
